File: main/elektrijada_22_23.kicad_sch (KiCad schematic)
At the start: 173 parts

Commit message: Updated schematics
Parts:
- R?: value R_Small -> 1k
Other:
- moved on the sheet: R?
Changed lines of the file:
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@@
     (stroke (width 0) (type default) (color 0 0 0 0))
   )
-  (wire (pts (xy 147.32 146.685) (xy 147.32 149.86))
+  (wire (pts (xy 147.32 146.685) (xy 147.32 148.59))
     (stroke (width 0) (type default) (color 0 0 0 0))
   )
@@
     (stroke (width 0) (type default) (color 0 0 0 0))
   )
-  (wire (pts (xy 147.32 163.195) (xy 147.32 162.56))
+  (wire (pts (xy 147.32 165.1) (xy 147.32 163.83))
     (stroke (width 0) (type default) (color 0 0 0 0))
   )
@@
     (stroke (width 0) (type default) (color 0 0 0 0))
   )
-  (wire (pts (xy 147.32 156.845) (xy 147.32 157.48))
+  (wire (pts (xy 147.32 156.845) (xy 147.32 158.75))
     (stroke (width 0) (type default) (color 0 0 0 0))
   )
@@
     (stroke (width 0) (type default) (color 0 0 0 0))
   )
-  (wire (pts (xy 147.32 154.94) (xy 147.32 156.845))
+  (wire (pts (xy 147.32 153.67) (xy 147.32 156.845))
     (stroke (width 0) (type default) (color 0 0 0 0))
   )
@@
       (effects (font (size 1.27 1.27)) hide)
     )
-    (pin "1")
-    (pin "2")
-    (pin "3")
-    (pin "5")
-    (pin "6")
-    (pin "7")
     (pin "4")
     (pin "8")
@@
       (effects (font (size 1.27 1.27)) hide)
     )
-    (pin "12")
-    (pin "13")
-    (pin "14")
-    (pin "15")
-    (pin "16")
-    (pin "10")
-    (pin "9")
     (pin "1")
     (pin "2")
@@
     (pin "4")
     (pin "5")
-    (pin "7")
-    (pin "8")
-    (pin "11")
-    (pin "6")
   )
   (symbol (lib_id "Device:R_Small") (at 46.99 148.59 90) (unit 1)
@@
       (effects (font (size 1.27 1.27)) hide)
     )
-    (pin "1")
-    (pin "2")
-    (pin "3")
-    (pin "4")
-    (pin "5")
-    (pin "6")
-    (pin "10")
-    (pin "11")
-    (pin "12")
-    (pin "13")
-    (pin "8")
-    (pin "9")
     (pin "14")
     (pin "7")
@@
     (pin "15")
     (pin "16")
-    (pin "10")
-    (pin "9")
-    (pin "1")
-    (pin "2")
-    (pin "3")
-    (pin "4")
-    (pin "5")
-    (pin "7")
-    (pin "8")
-    (pin "11")
-    (pin "6")
   )
   (symbol (lib_id "Device:C_Polarized_Small") (at 144.145 208.28 0) (unit 1)
@@
     (pin "2")
   )
-  (symbol (lib_id "power:GND") (at 147.32 163.195 0) (unit 1)
+  (symbol (lib_id "power:GND") (at 147.32 165.1 0) (unit 1)
     (in_bom yes) (on_board yes)
-    (property "Reference" "#PWR?" (id 0) (at 147.32 169.545 0)
+    (property "Reference" "#PWR?" (id 0) (at 147.32 171.45 0)
       (effects (font (size 1.27 1.27)) hide)
     )
-    (property "Value" "GND" (id 1) (at 149.86 166.37 0))
-    (property "Footprint" "" (id 2) (at 147.32 163.195 0)
+    (property "Value" "GND" (id 1) (at 149.86 168.275 0))
+    (property "Footprint" "" (id 2) (at 147.32 165.1 0)
       (effects (font (size 1.27 1.27)) hide)
     )
-    (property "Datasheet" "" (id 3) (at 147.32 163.195 0)
+    (property "Datasheet" "" (id 3) (at 147.32 165.1 0)
       (effects (font (size 1.27 1.27)) hide)
     )
@@
       (effects (font (size 1.27 1.27)) hide)
     )
-    (pin "1")
-    (pin "2")
-    (pin "3")
     (pin "5")
     (pin "6")
     (pin "7")
-    (pin "4")
-    (pin "8")
   )
   (symbol (lib_id "Device:R_Small") (at 229.87 36.195 0) (unit 1)
@@
       (effects (font (size 1.27 1.27)) hide)
     )
-    (pin "1")
-    (pin "2")
-    (pin "3")
     (pin "5")
     (pin "6")
     (pin "7")
-    (pin "4")
-    (pin "8")
   )
   (symbol (lib_id "Amplifier_Operational:TL072") (at 33.02 196.85 0) (unit 1)
@@
     (pin "2")
     (pin "3")
-    (pin "5")
-    (pin "6")
-    (pin "7")
-    (pin "4")
-    (pin "8")
   )
   (symbol (lib_id "power:GND") (at 348.615 33.655 0) (unit 1)
@@
       (effects (font (size 1.27 1.27)) hide)
     )
-    (pin "1")
-    (pin "2")
-    (pin "3")
     (pin "5")
     (pin "6")
     (pin "7")
-    (pin "4")
-    (pin "8")
   )
   (symbol (lib_id "Power_Protection:USBLC6-2SC6") (at 300.99 54.61 0) (unit 1)
@@
       (effects (font (size 1.27 1.27)) hide)
     )
-    (pin "1")
-    (pin "2")
-    (pin "3")
     (pin "5")
     (pin "6")
     (pin "7")
-    (pin "4")
-    (pin "8")
   )
   (symbol (lib_id "Device:R_Potentiometer_Small") (at 154.94 106.045 90) (mirror x) (unit 1)
@@
       (effects (font (size 1.27 1.27)) hide)
     )
-    (pin "1")
-    (pin "2")
-    (pin "3")
     (pin "4")
     (pin "5")
@@
       (effects (font (size 1.27 1.27)) hide)
     )
-    (pin "1")
-    (pin "2")
-    (pin "3")
-    (pin "4")
-    (pin "5")
-    (pin "6")
     (pin "10")
     (pin "11")
@@
     (pin "8")
     (pin "9")
-    (pin "14")
-    (pin "7")
   )
   (symbol (lib_id "power:GND") (at 391.16 65.405 0) (unit 1)
@@
     (in_bom yes) (on_board yes) (fields_autoplaced)
     (property "Reference" "R?" (id 0) (at 80.01 187.96 90))
-    (property "Value" "R_Small" (id 1) (at 80.01 190.5 90))
+    (property "Value" "1k" (id 1) (at 80.01 190.5 90))
     (property "Footprint" "" (id 2) (at 80.01 194.31 0)
       (effects (font (size 1.27 1.27)) hide)
@@
     (pin "2")
     (pin "3")
-    (pin "5")
-    (pin "6")
-    (pin "7")
-    (pin "4")
-    (pin "8")
   )
   (symbol (lib_id "Device:R_Small") (at 220.345 39.37 0) (unit 1)
@@
     (pin "1")
   )
-  (symbol (lib_id "Device:R_Small") (at 147.32 160.02 0) (unit 1)
+  (symbol (lib_id "Device:R_Small") (at 147.32 161.29 0) (unit 1)
     (in_bom yes) (on_board yes) (fields_autoplaced)
-    (property "Reference" "R?" (id 0) (at 149.225 158.7499 0)
+    (property "Reference" "R?" (id 0) (at 149.225 160.0199 0)
       (effects (font (size 1.27 1.27)) (justify left))
     )
-    (property "Value" "2k" (id 1) (at 149.225 161.2899 0)
+    (property "Value" "2k" (id 1) (at 149.225 162.5599 0)
       (effects (font (size 1.27 1.27)) (justify left))
     )
-    (property "Footprint" "" (id 2) (at 147.32 160.02 0)
+    (property "Footprint" "" (id 2) (at 147.32 161.29 0)
       (effects (font (size 1.27 1.27)) hide)
     )
-    (property "Datasheet" "~" (id 3) (at 147.32 160.02 0)
+    (property "Datasheet" "~" (id 3) (at 147.32 161.29 0)
       (effects (font (size 1.27 1.27)) hide)
     )
@@
     (pin "2")
     (pin "3")
-    (pin "4")
-    (pin "5")
-    (pin "6")
   )
   (symbol (lib_id "Device:R_Small") (at 64.135 82.55 0) (unit 1)
@@
     (pin "2")
     (pin "3")
-    (pin "5")
-    (pin "6")
-    (pin "7")
-    (pin "4")
-    (pin "8")
   )
   (symbol (lib_id "Device:R_Small") (at 169.545 31.75 0) (unit 1)
@@
       (effects (font (size 1.27 1.27)) hide)
     )
-    (pin "1")
-    (pin "2")
-    (pin "3")
-    (pin "5")
-    (pin "6")
-    (pin "7")
     (pin "4")
     (pin "8")
@@
       (effects (font (size 1.27 1.27)) hide)
     )
-    (pin "1")
-    (pin "2")
-    (pin "3")
-    (pin "5")
-    (pin "6")
-    (pin "7")
     (pin "4")
     (pin "8")
@@
       (effects (font (size 1.27 1.27)) hide)
     )
-    (pin "1")
-    (pin "2")
-    (pin "3")
-    (pin "5")
-    (pin "6")
-    (pin "7")
     (pin "4")
     (pin "8")
@@
     (pin "2")
     (pin "3")
-    (pin "5")
-    (pin "6")
-    (pin "7")
-    (pin "4")
-    (pin "8")
   )
   (symbol (lib_id "Device:C_Small") (at 40.005 241.935 0) (unit 1)
@@
     (pin "5")
     (pin "6")
-    (pin "10")
-    (pin "11")
-    (pin "12")
-    (pin "13")
-    (pin "8")
-    (pin "9")
-    (pin "14")
-    (pin "7")
   )
   (symbol (lib_id "Device:C_Small") (at 220.345 54.61 0) (unit 1)
@@
       (effects (font (size 1.27 1.27)) hide)
     )
-    (pin "12")
-    (pin "13")
-    (pin "14")
-    (pin "15")
-    (pin "16")
-    (pin "10")
-    (pin "9")
-    (pin "1")
-    (pin "2")
-    (pin "3")
-    (pin "4")
-    (pin "5")
     (pin "7")
     (pin "8")
-    (pin "11")
-    (pin "6")
   )
   (symbol (lib_id "power:GND") (at 83.185 25.4 90) (unit 1)
@@
       (effects (font (size 1.27 1.27)) hide)
     )
-    (pin "12")
-    (pin "13")
-    (pin "14")
-    (pin "15")
-    (pin "16")
-    (pin "10")
-    (pin "9")
-    (pin "1")
-    (pin "2")
-    (pin "3")
-    (pin "4")
-    (pin "5")
-    (pin "7")
-    (pin "8")
     (pin "11")
     (pin "6")
@@
     (pin "1")
   )
-  (symbol (lib_id "Device:R_Small") (at 147.32 152.4 0) (unit 1)
+  (symbol (lib_id "Device:R_Small") (at 147.32 151.13 0) (unit 1)
     (in_bom yes) (on_board yes) (fields_autoplaced)
-    (property "Reference" "R?" (id 0) (at 149.225 151.1299 0)
+    (property "Reference" "R?" (id 0) (at 149.225 149.8599 0)
       (effects (font (size 1.27 1.27)) (justify left))
     )
-    (property "Value" "2k" (id 1) (at 149.225 153.6699 0)
+    (property "Value" "2k" (id 1) (at 149.225 152.3999 0)
       (effects (font (size 1.27 1.27)) (justify left))
     )
-    (property "Footprint" "" (id 2) (at 147.32 152.4 0)
+    (property "Footprint" "" (id 2) (at 147.32 151.13 0)
       (effects (font (size 1.27 1.27)) hide)
     )
-    (property "Datasheet" "~" (id 3) (at 147.32 152.4 0)
+    (property "Datasheet" "~" (id 3) (at 147.32 151.13 0)
       (effects (font (size 1.27 1.27)) hide)
     )
@@
       (effects (font (size 1.27 1.27)) hide)
     )
-    (pin "12")
-    (pin "13")
-    (pin "14")
-    (pin "15")
-    (pin "16")
     (pin "10")
     (pin "9")
-    (pin "1")
-    (pin "2")
-    (pin "3")
-    (pin "4")
-    (pin "5")
-    (pin "7")
-    (pin "8")
-    (pin "11")
-    (pin "6")
   )
   (symbol (lib_id "Device:R_Small") (at 142.875 253.365 180) (unit 1)
@@
     )
     (path "/59d4af11-137a-4bf7-92e7-f33b9b93bf0a"
-      (reference "R?") (unit 1) (value "R_Small") (footprint "")
+      (reference "R?") (unit 1) (value "1k") (footprint "")
     )
     (path "/5e953da8-a313-4290-ae9c-2cb115f28d55"

Commit message: Chore: USB interface schematic
Parts:
- added C?: 100n, symbol Device:C_Small
- added C?: 10u, symbol Device:C_Polarized_Small
- added R? (x2): 22R, symbol Device:R_Small
- added U?: LD1117, Package_TO_SOT_SMD:SOT-223-3_TabPin2, symbol Regulator_Linear:LD1117S18TR_SOT223
- C? (x35), D? (x15), J? (x3), JP? (x4), L?, Q? (x12), R? (x68), RV? (x10), U? (x25): Manufacturer (none) -> -; Order Code (none) -> -; Part Number (none) -> -; Supplier (none) -> -
Connections:
- net +5V: now also U?.3 (VBUS), U?.9 (SEL1), C?.1, U?.3 (VI)
- net D+: now also R?.2; no longer U?.1 (I/O1)
- net D-: now also R?.2; no longer U?.3 (I/O2)
- net GND: now also U?.4 (DGNDU), C?.2, C?.2, U?.1 (GND)
- net VDD: now reaches U?.10 (VCCC)
- net VDD: now also C?.1, U?.2 (VO)
- new net Dres+: R?.1, U?.1 (I/O1)
- new net Dres-: R?.1, U?.3 (I/O2)
- no-connect marks 3 -> 6
Other:
- moved on the sheet: U?

Commit message: Chore: USB interface design
Parts:
- added C?: 10u, symbol Device:C_Polarized_Small
- added C?: 100n, symbol Device:C_Small
- added U?: LD1117, Package_TO_SOT_SMD:SOT-223-3_TabPin2, symbol Regulator_Linear:LD1117S18TR_SOT223
Connections:
- net +5V: now also C?.1, U?.3 (VI); no longer U?.3 (VBUS)
- net GND: now also U?.18 (AGNDP), U?.21 (XTI), U?.22 (AGNDX), U?.26 (DGND), C?.2, C?.2, U?.1 (GND)
- net VDD: now also U?.3 (VBUS); no longer U?.10 (VCCC)
- net VDDA: now reaches U?.17 (VCCP1)
- net VDDA: now also U?.10 (VCCC), U?.23 (VCCX), C?.1, U?.2 (VO)
- no-connect marks 6 -> 8

Commit message: Chore: USB interface
Connections:
- net GND: now also U?.11 (AGNDC)
Changed lines of the file:
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@@
     (stroke (width 0) (type default) (color 0 0 0 0))
   )
+  (wire (pts (xy 302.26 133.35) (xy 304.8 133.35))
+    (stroke (width 0) (type default) (color 0 0 0 0))
+  )
   (wire (pts (xy 277.495 256.54) (xy 277.495 259.08))
     (stroke (width 0) (type default) (color 0 0 0 0))
@@
       (effects (font (size 1.27 1.27)) hide)
     )
+    (pin "1")
+    (pin "2")
+    (pin "3")
+    (pin "5")
+    (pin "6")
+    (pin "7")
     (pin "4")
     (pin "8")
@@
       (effects (font (size 1.27 1.27)) hide)
     )
+    (pin "12")
+    (pin "13")
+    (pin "14")
+    (pin "15")
+    (pin "16")
+    (pin "10")
+    (pin "9")
     (pin "1")
     (pin "2")
@@
     (pin "4")
     (pin "5")
+    (pin "7")
+    (pin "8")
+    (pin "11")
+    (pin "6")
   )
   (symbol (lib_id "Device:R_Small") (at 46.99 148.59 90) (unit 1)
@@
       (effects (font (size 1.27 1.27)) hide)
     )
+    (pin "1")
+    (pin "2")
+    (pin "3")
+    (pin "4")
+    (pin "5")
+    (pin "6")
+    (pin "10")
+    (pin "11")
+    (pin "12")
+    (pin "13")
+    (pin "8")
+    (pin "9")
     (pin "14")
     (pin "7")
@@
     (pin "15")
     (pin "16")
+    (pin "10")
+    (pin "9")
+    (pin "1")
+    (pin "2")
+    (pin "3")
+    (pin "4")
+    (pin "5")
+    (pin "7")
+    (pin "8")
+    (pin "11")
+    (pin "6")
   )
   (symbol (lib_id "Device:C_Polarized_Small") (at 144.145 208.28 0) (unit 1)
@@
       (effects (font (size 1.27 1.27)) hide)
     )
+    (pin "1")
+    (pin "2")
+    (pin "3")
     (pin "5")
     (pin "6")
     (pin "7")
+    (pin "4")
+    (pin "8")
   )
   (symbol (lib_id "Device:R_Small") (at 229.87 36.195 0) (unit 1)
@@
       (effects (font (size 1.27 1.27)) hide)
     )
+    (pin "1")
+    (pin "2")
+    (pin "3")
     (pin "5")
     (pin "6")
     (pin "7")
+    (pin "4")
+    (pin "8")
   )
   (symbol (lib_id "Amplifier_Operational:TL072") (at 33.02 196.85 0) (unit 1)
@@
     (pin "2")
     (pin "3")
+    (pin "5")
+    (pin "6")
+    (pin "7")
+    (pin "4")
+    (pin "8")
   )
   (symbol (lib_id "power:GND") (at 348.615 33.655 0) (unit 1)
@@
       (effects (font (size 1.27 1.27)) hide)
     )
+    (pin "1")
+    (pin "2")
+    (pin "3")
     (pin "5")
     (pin "6")
     (pin "7")
+    (pin "4")
+    (pin "8")
   )
   (symbol (lib_id "Power_Protection:USBLC6-2SC6") (at 307.34 45.72 0) (unit 1)
@@
       (effects (font (size 1.27 1.27)) hide)
     )
+    (pin "1")
+    (pin "2")
+    (pin "3")
     (pin "5")
     (pin "6")
     (pin "7")
+    (pin "4")
+    (pin "8")
   )
   (symbol (lib_id "power:VDD") (at 302.26 113.03 90) (unit 1)
@@
       (effects (font (size 1.27 1.27)) hide)
     )
+    (pin "1")
+    (pin "2")
+    (pin "3")
     (pin "4")
     (pin "5")
@@
       (effects (font (size 1.27 1.27)) hide)
     )
+    (pin "1")
+    (pin "2")
+    (pin "3")
+    (pin "4")
+    (pin "5")
+    (pin "6")
     (pin "10")
     (pin "11")
@@
     (pin "8")
     (pin "9")
+    (pin "14")
+    (pin "7")
   )
   (symbol (lib_id "power:GND") (at 391.16 65.405 0) (unit 1)
@@
     (pin "2")
     (pin "3")
+    (pin "5")
+    (pin "6")
+    (pin "7")
+    (pin "4")
+    (pin "8")
   )
   (symbol (lib_id "power:+5V") (at 302.26 128.27 90) (unit 1)
@@
     (pin "2")
     (pin "3")
+    (pin "4")
+    (pin "5")
+    (pin "6")
   )
   (symbol (lib_id "Device:R_Small") (at 64.135 82.55 0) (unit 1)
@@
     (pin "2")
     (pin "3")
+    (pin "5")
+    (pin "6")
+    (pin "7")
+    (pin "4")
+    (pin "8")
   )
   (symbol (lib_id "power:+5V") (at 288.29 230.505 0) (unit 1)
@@
       (effects (font (size 1.27 1.27)) hide)
     )
+    (pin "1")
+    (pin "2")
+    (pin "3")
+    (pin "5")
+    (pin "6")
+    (pin "7")
     (pin "4")
     (pin "8")
@@
       (effects (font (size 1.27 1.27)) hide)
     )
+    (pin "1")
+    (pin "2")
+    (pin "3")
+    (pin "5")
+    (pin "6")
+    (pin "7")
     (pin "4")
     (pin "8")
@@
       (effects (font (size 1.27 1.27)) hide)
     )
+    (pin "1")
+    (pin "2")
+    (pin "3")
+    (pin "5")
+    (pin "6")
+    (pin "7")
     (pin "4")
     (pin "8")
@@
     (pin "2")
     (pin "3")
+    (pin "5")
+    (pin "6")
+    (pin "7")
+    (pin "4")
+    (pin "8")
   )
   (symbol (lib_id "Device:C_Small") (at 40.005 241.935 0) (unit 1)
@@
     (pin "5")
     (pin "6")
+    (pin "10")
+    (pin "11")
+    (pin "12")
+    (pin "13")
+    (pin "8")
+    (pin "9")
+    (pin "14")
+    (pin "7")
   )
   (symbol (lib_id "Device:C_Small") (at 220.345 54.61 0) (unit 1)
@@
       (effects (font (size 1.27 1.27)) hide)
     )
+    (pin "12")
+    (pin "13")
+    (pin "14")
+    (pin "15")
+    (pin "16")
+    (pin "10")
+    (pin "9")
+    (pin "1")
+    (pin "2")
+    (pin "3")
+    (pin "4")
+    (pin "5")
     (pin "7")
     (pin "8")
+    (pin "11")
+    (pin "6")
   )
   (symbol (lib_id "power:GND") (at 83.185 25.4 90) (unit 1)
@@
       (effects (font (size 1.27 1.27)) hide)
     )
+    (pin "12")
+    (pin "13")
+    (pin "14")
+    (pin "15")
+    (pin "16")
+    (pin "10")
+    (pin "9")
+    (pin "1")
+    (pin "2")
+    (pin "3")
+    (pin "4")
+    (pin "5")
+    (pin "7")
+    (pin "8")
     (pin "11")
     (pin "6")
@@
       (effects (font (size 1.27 1.27)) hide)
     )
+    (pin "12")
+    (pin "13")
+    (pin "14")
+    (pin "15")
+    (pin "16")
     (pin "10")
     (pin "9")
+    (pin "1")
+    (pin "2")
+    (pin "3")
+    (pin "4")
+    (pin "5")
+    (pin "7")
+    (pin "8")
+    (pin "11")
+    (pin "6")
   )
   (symbol (lib_id "Device:R_Small") (at 142.875 253.365 180) (unit 1)
