File: addon/LT1618/LT1618.kicad_pcb (KiCad board)
At the start: 2 copper layers, 40 x 15.2 mm, 14 parts, among them J1 Conn_01x04, J2 Conn_01x04, U1 LT1618

Commit message: Fix: changed out inductor and flipped pin headers
Parts:
- J1, J2: moved to B.Cu
- L1: footprint Inductor_THT:L_Radial_D7.2mm_P3.00mm_Murata_1700 -> Inductor_SMD:L_Bourns_SRN6045TA
- moved L1 1.87 mm to (171.6, 91.6)
- turned J1 to 180 degrees
- turned J2 to 180 degrees
Connections:
- net Net-(D1-Pad2) renamed /ind_fill
Routing:
- net /ind_fill: track 11.6 -> 3.35 mm
- net Net-(L1-Pad1): track 12.8 -> 13.4 mm
- added copper zone on F.Cu, net /ind_fill
